Commit message: Working rover simulation with RPLIDAR A1

File: src/rover_description/urdf/rover.urdf (robot description, URDF)
Before this commit: robot robot, 9 links, 8 joints
Links:
- link front_left_wheel: geometry collision cylinder length=0.04 radius=0.035; visual cylinder length=0.04 radius=0.035
- link front_right_wheel: geometry collision cylinder length=0.04 radius=0.035; visual cylinder length=0.04 radius=0.035
- link lidar_link: mass 0.1 -> 0.17; geometry collision cylinder length=0.042 radius=0.048; visual cylinder length=0.005 radius=0.03
- link rear_left_wheel: geometry collision cylinder length=0.04 radius=0.035; visual cylinder length=0.04 radius=0.035
- link rear_right_wheel: geometry collision cylinder length=0.04 radius=0.035; visual cylinder length=0.04 radius=0.035
Joints:
- joint lidar_joint: origin xyz=0 0 0.07022 rpy=0 0 0 -> xyz=0 0 0.08522 rpy=0 0 0

File: src/rover_description/urdf/rover.xacro (robot description, xacro)
@@ -18,4 +18,9 @@
 <xacro:property name="camera_y" value="0"/>                <!-- Centered -->
 <xacro:property name="camera_z" value="${b/4}"/>           <!-- Half height of rover -->
+<!-- RPLIDAR A1 Dimensions - CORRECTED HEIGHT -->
+<xacro:property name="lidar_height" value="0.042"/>        <!-- RPLIDAR A1 height (42mm) -->
+<xacro:property name="lidar_radius" value="0.048"/>        <!-- RPLIDAR A1 radius (48mm) -->
+<!-- Lidar at 0.15m above base_link to intersect obstacles at z=0.25-0.75 -->
+<xacro:property name="lidar_mount_z" value="0.20"/>
 <!-- Material Density -->
 <xacro:property name="d1" value="2710.0"/>   <!-- body (aluminium) -->
@@ -31,8 +36,17 @@
 <xacro:property name="Iz_wheel" value="${0.5*m2*r*r}"/>
 <xacro:property name="I_wheel"  value="${(1.0/12.0)*m2*(3.0*r*r+d*d)}"/>
-<!-- Materials for visualization -->
-<xacro:property name="body_color" value="0.8 0.2 0.2 1.0"/>   <!-- Red -->
-<xacro:property name="wheel_color" value="0.2 0.2 0.2 1.0"/>  <!-- Dark grey -->
-<xacro:property name="camera_color" value="0.1 0.1 0.3 1.0"/> <!-- Dark blue -->
+<!-- ============================================================== -->
+<!-- PREMIUM COLORS                                                -->
+<!-- ============================================================== -->
+<xacro:property name="body_color" value="0.02 0.02 0.02 1.0"/>           <!-- Deep Black -->
+<xacro:property name="body_metallic" value="0.05 0.05 0.05 1.0"/>        <!-- Satin Black -->
+<!-- LIDAR - Deep Metallic Burgundy -->
+<xacro:property name="lidar_color" value="0.35 0.05 0.08 1.0"/>          <!-- Deep Burgundy -->
+<xacro:property name="lidar_top_color" value="0.12 0.12 0.12 1.0"/>      <!-- Dark Gunmetal -->
+<!-- CAMERA - Bold Premium Blue -->
+<xacro:property name="camera_color" value="0.05 0.25 0.65 1.0"/>         <!-- Bold Premium Blue -->
+<!-- WHEELS - Premium Dark Alloy -->
+<xacro:property name="wheel_color" value="0.08 0.08 0.08 1.0"/>          <!-- Dark Alloy -->
+<xacro:property name="wheel_rim_color" value="0.85 0.85 0.88 1.0"/>      <!-- Premium Silver -->
 <!-- Inertia macro: body -->
 <xacro:macro name="inertia_body">
@@ -46,5 +60,4 @@
 </xacro:macro>
 <!-- Inertia macro: wheel -->
-<!-- rpy="1.5708 0 0" rotates the inertia tensor to match cylinder lying on its side -->
 <xacro:macro name="inertia_wheel">
     <inertial>
@@ -56,7 +69,6 @@
     </inertial>
 </xacro:macro>
-<!-- ========== BASE FOOTPRINT ========== -->
+<!-- ========== BASE ========== -->
 <link name="base_footprint"/>
-<!-- ========== BASE TO FOOTPRINT JOINT ========== -->
 <joint name="base_joint" type="fixed">
     <parent link="base_footprint"/>
@@ -84,7 +96,7 @@
 </link>
 <!-- ============================================================== -->
-<!-- WHEELS (Using ROS Convention: +X=Front, +Y=Left, +Z=Up)        -->
-<!-- ============================================================== -->
-<!-- ========== FRONT LEFT WHEEL ========== -->
+<!-- WHEELS                                                         -->
+<!-- ============================================================== -->
+<!-- FRONT LEFT WHEEL -->
 <joint name="front_left_wheel_joint" type="continuous">
     <parent link="base_link"/>
@@ -96,5 +108,5 @@
 </joint>
 <link name="front_left_wheel">
-    <visual>
+    <visual name="tire">
         <origin rpy="1.5708 0 0" xyz="0 0 0"/>
         <geometry>
@@ -105,4 +117,13 @@
         </material>
     </visual>
+    <visual name="rim">
+        <origin rpy="1.5708 0 0" xyz="0 0 0"/>
+        <geometry>
+            <cylinder length="${d + 0.002}" radius="${r * 0.65}"/>
+        </geometry>
+        <material name="wheel_rim_material">
+            <color rgba="${wheel_rim_color}"/>
+        </material>
+    </visual>
     <collision>
         <origin rpy="1.5708 0 0" xyz="0 0 0"/>
@@ -113,5 +134,5 @@
     <xacro:inertia_wheel/>
 </link>
-<!-- ========== FRONT RIGHT WHEEL ========== -->
+<!-- FRONT RIGHT WHEEL -->
 <joint name="front_right_wheel_joint" type="continuous">
     <parent link="base_link"/>
@@ -123,5 +144,5 @@
 </joint>
 <link name="front_right_wheel">
-    <visual>
+    <visual name="tire">
         <origin rpy="1.5708 0 0" xyz="0 0 0"/>
         <geometry>
@@ -132,4 +153,13 @@
         </material>
     </visual>
+    <visual name="rim">
+        <origin rpy="1.5708 0 0" xyz="0 0 0"/>
+        <geometry>
+            <cylinder length="${d + 0.002}" radius="${r * 0.65}"/>
+        </geometry>
+        <material name="wheel_rim_material">
+            <color rgba="${wheel_rim_color}"/>
+        </material>
+    </visual>
     <collision>
         <origin rpy="1.5708 0 0" xyz="0 0 0"/>
@@ -140,5 +170,5 @@
     <xacro:inertia_wheel/>
 </link>
-<!-- ========== REAR LEFT WHEEL ========== -->
+<!-- REAR LEFT WHEEL -->
 <joint name="rear_left_wheel_joint" type="continuous">
     <parent link="base_link"/>
@@ -150,5 +180,5 @@
 </joint>
 <link name="rear_left_wheel">
-    <visual>
+    <visual name="tire">
         <origin rpy="1.5708 0 0" xyz="0 0 0"/>
         <geometry>
@@ -159,4 +189,13 @@
         </material>
     </visual>
+    <visual name="rim">
+        <origin rpy="1.5708 0 0" xyz="0 0 0"/>
+        <geometry>
+            <cylinder length="${d + 0.002}" radius="${r * 0.65}"/>
+        </geometry>
+        <material name="wheel_rim_material">
+            <color rgba="${wheel_rim_color}"/>
+        </material>
+    </visual>
     <collision>
         <origin rpy="1.5708 0 0" xyz="0 0 0"/>
@@ -167,5 +206,5 @@
     <xacro:inertia_wheel/>
 </link>
-<!-- ========== REAR RIGHT WHEEL ========== -->
+<!-- REAR RIGHT WHEEL -->
 <joint name="rear_right_wheel_joint" type="continuous">
     <parent link="base_link"/>
@@ -177,5 +216,5 @@
 </joint>
 <link name="rear_right_wheel">
-    <visual>
+    <visual name="tire">
         <origin rpy="1.5708 0 0" xyz="0 0 0"/>
         <geometry>
@@ -186,4 +225,13 @@
         </material>
     </visual>
+    <visual name="rim">
+        <origin rpy="1.5708 0 0" xyz="0 0 0"/>
+        <geometry>
+            <cylinder length="${d + 0.002}" radius="${r * 0.65}"/>
+        </geometry>
+        <material name="wheel_rim_material">
+            <color rgba="${wheel_rim_color}"/>
+        </material>
+    </visual>
     <collision>
         <origin rpy="1.5708 0 0" xyz="0 0 0"/>
@@ -195,7 +243,6 @@
 </link>
 <!-- ============================================================== -->
-<!-- RPI CAMERA - MOUNTED ON FRONT FACE LOOKING FORWARD            -->
-<!-- ============================================================== -->
-<!-- Camera mount joint (physical camera on front face) -->
+<!-- RPI CAMERA                                                     -->
+<!-- ============================================================== -->
 <joint name="camera_joint" type="fixed">
     <parent link="base_link"/>
@@ -203,5 +250,4 @@
     <origin xyz="${camera_x} ${camera_y} ${camera_z}" rpy="0 1.5708 0"/>
 </joint>
-<!-- Camera physical link -->
 <link name="camera_link">
     <visual>
@@ -228,8 +274,4 @@
     </inertial>
 </link>
-<!-- Optical frame joint (for camera sensor) -->
-<!-- This represents the actual camera sensor frame looking forward -->
-<!-- rpy="0 -1.5708 0" rotates camera to look forward (+X direction) -->
-<!-- Then rpy="-1.5708 0 -1.5708" aligns Z forward for optical convention -->
 <joint name="camera_optical_joint" type="fixed">
     <parent link="camera_link"/>
@@ -237,37 +279,49 @@
     <origin xyz="0 0 0.0045" rpy="-1.5708 0 -1.5708"/>
 </joint>
-<!-- Optical frame link -->
-<!-- This follows REP-103/REP-104 standard for camera frames -->
-<!-- Z is forward (optical axis), X is right, Y is down -->
 <link name="camera_optical_frame"/>
-<!--LIDAR-->
-<!-- ============================================================== -->
-<!-- LIDAR WITH FULL GAZEBO CONFIGURATION                          -->
-<!-- ============================================================== -->
-<!-- Lidar mount joint -->
+<!-- ============================================================== -->
+<!-- RPLIDAR A1 - FIXED HEIGHT                                      -->
+<!-- ============================================================== -->
+<!-- ============================================================== -->
+<!-- RPLIDAR A1 - CORRECTED HEIGHT                                  -->
+<!-- ============================================================== -->
+<!-- Lidar joint - mounted higher -->
+<!-- ============================================================== -->
+<!-- RPLIDAR A1 - CORRECTED: NOT HOVERING, RAYS FROM MIDDLE        -->
+<!-- ============================================================== -->
+<!-- Lidar joint - mounted just above the rover body -->
 <joint name="lidar_joint" type="fixed">
-    <origin xyz="0 0 ${b/2 + 0.01}" rpy="0 0 0"/>
+    <origin xyz="0 0 ${b/2 + 0.015}" rpy="0 0 0"/>  <!-- Just above body -->
     <parent link="base_link"/>
     <child link="lidar_link"/>
 </joint>
-<!-- Lidar base link -->
+<!-- Lidar visual -->
 <link name="lidar_link">
-    <visual>
-        <origin xyz="0 0 0" rpy="0 0 0"/>
-        <geometry>
-            <cylinder length="0.03" radius="0.055"/>
+    <visual name="lidar_body">
+        <origin rpy="0 0 0" xyz="0 0 0"/>
+        <geometry>
+            <cylinder length="${lidar_height}" radius="${lidar_radius}"/>
         </geometry>
         <material name="lidar_material">
-            <color rgba="0.1 0.8 0.1 1.0"/>
-        </material>
-    </visual>
-    <collision>
-        <origin xyz="0 0 0" rpy="0 0 0"/>
-        <geometry>
-            <cylinder length="0.03" radius="0.055"/>
+            <color rgba="${lidar_color}"/>
+        </material>
+    </visual>
+    <visual name="lidar_top">
+        <origin rpy="0 0 0" xyz="0 0 ${lidar_height/2 - 0.005}"/>
+        <geometry>
+            <cylinder length="0.005" radius="0.03"/>
+        </geometry>
+        <material name="lidar_top_material">
+            <color rgba="${lidar_top_color}"/>
+        </material>
+    </visual>
+    <collision>
+        <origin rpy="0 0 0" xyz="0 0 0"/>
+        <geometry>
+            <cylinder length="${lidar_height}" radius="${lidar_radius}"/>
         </geometry>
     </collision>
     <inertial>
-        <mass value="0.1"/>
+        <mass value="0.17"/>
         <origin xyz="0 0 0" rpy="0 0 0"/>
         <inertia ixx="0.0001" ixy="0" ixz="0"
@@ -276,70 +330,32 @@
     </inertial>
 </link>
-<!-- Lidar spinner joint (continuous rotation) -->
-<joint name="lidar_spinner_joint" type="continuous">
-    <parent link="lidar_link"/>
-    <child link="lidar_spinner_link"/>
-    <origin xyz="0 0 0.015" rpy="0 0 0"/>
-    <axis xyz="0 0 1"/>
-    <limit effort="10.0" velocity="10.0"/>
-    <dynamics damping="0.1" friction="0.1"/>
-</joint>
-<!-- Lidar spinner link -->
-<link name="lidar_spinner_link">
-    <visual>
-        <origin xyz="0 0 0" rpy="0 0 0"/>
-        <geometry>
-            <cylinder length="0.015" radius="0.04"/>
-        </geometry>
-        <material name="lidar_spinner_material">
-            <color rgba="0.1 0.5 0.1 1.0"/>
-        </material>
-    </visual>
-    <collision>
-        <origin xyz="0 0 0" rpy="0 0 0"/>
-        <geometry>
-            <cylinder length="0.015" radius="0.04"/>
-        </geometry>
-    </collision>
-    <inertial>
-        <mass value="0.05"/>
-        <origin xyz="0 0 0" rpy="0 0 0"/>
-        <inertia ixx="0.00001" ixy="0" ixz="0"
-                 iyy="0.00001" iyz="0"
-                 izz="0.00001"/>
-    </inertial>
-</link>
-<!-- Lidar sensor frame -->
-<joint name="lidar_sensor_joint" type="fixed">
-    <parent link="lidar_spinner_link"/>
-    <child link="lidar_sensor_frame"/>
-    <origin xyz="0 0 0.01" rpy="0 0 0"/>
-</joint>
-<link name="lidar_sensor_frame"/>
-<!-- ============================================================== -->
-<!-- GAZEBO LIDAR PLUGIN CONFIGURATION                             -->
-<!-- ============================================================== -->
-<gazebo reference="lidar_sensor_frame">
-    <sensor type="ray" name="lidar_sensor">
-        <pose>0 0 0 0 0 0</pose>
+<!-- ============================================================== -->
+<!-- GAZEBO LIDAR SENSOR - RAYS FROM MIDDLE OF LIDAR               -->
+<!-- ============================================================== -->
+<gazebo reference="lidar_link">
+    <sensor name="gpu_lidar" type="gpu_lidar">
+        <!-- Rays from the center of the lidar (NOT the top) -->
+        <pose>0 0 ${lidar_height/4} 0 0 0</pose>
+        <always_on>true</always_on>
         <visualize>true</visualize>
-        <update_rate>10.0</update_rate>
-        <ray>
+        <update_rate>10</update_rate>
+        <topic>scan</topic>
+        <lidar>
             <scan>
                 <horizontal>
-                    <samples>360</samples>
-                    <resolution>1.0</resolution>      <!-- 1 degree resolution -->
-                    <min_angle>-3.14159265</min_angle> <!-- -180 degrees -->
-                    <max_angle>3.14159265</max_angle>  <!-- +180 degrees -->
+                    <samples>720</samples>
+                    <resolution>1</resolution>
+                    <min_angle>-3.14159</min_angle>
+                    <max_angle>3.14159</max_angle>
                 </horizontal>
                 <vertical>
                     <samples>1</samples>
-                    <resolution>0.0</resolution>
-                    <min_angle>0.0</min_angle>
-                    <max_angle>0.0</max_angle>
+                    <resolution>0.01</resolution>
+                    <min_angle>0</min_angle>
+                    <max_angle>0</max_angle>
                 </vertical>
             </scan>
             <range>
-                <min>0.1</min>
+                <min>0.05</min>
                 <max>12.0</max>
                 <resolution>0.01</resolution>
@@ -348,16 +364,58 @@
                 <type>gaussian</type>
                 <mean>0.0</mean>
-                <stddev>0.01</stddev>
+                <stddev>0.001</stddev>
             </noise>
-        </ray>
-        <plugin name="lidar_controller" filename="libgazebo_ros_ray_sensor.so">
-            <ros>
-                <namespace>/</namespace>
-                <remapping>~/out:=/scan</remapping>
-            </ros>
-            <frame_name>lidar_sensor_frame</frame_name>
-            <topic_name>/scan</topic_name>
-        </plugin>
+        </lidar>
     </sensor>
 </gazebo>
+<!-- ============================================================== -->
+<!-- GAZEBO CONFIGURATIONS                                          -->
+<!-- ============================================================== -->
+<gazebo reference="front_left_wheel">
+    <mu1>0.8</mu1>
+    <mu2>0.05</mu2>
+    <kp>1000000.0</kp>
+    <kd>100.0</kd>
+    <minDepth>0.001</minDepth>
+    <material>Gazebo/DarkGrey</material>
+</gazebo>
+<gazebo reference="front_right_wheel">
+    <mu1>0.8</mu1>
+    <mu2>0.05</mu2>
+    <kp>1000000.0</kp>
+    <kd>100.0</kd>
+    <minDepth>0.001</minDepth>
+    <material>Gazebo/DarkGrey</material>
+</gazebo>
+<gazebo reference="rear_left_wheel">
+    <mu1>0.8</mu1>
+    <mu2>0.05</mu2>
+    <kp>1000000.0</kp>
+    <kd>100.0</kd>
+    <minDepth>0.001</minDepth>
+    <material>Gazebo/DarkGrey</material>
+</gazebo>
+<gazebo reference="rear_right_wheel">
+    <mu1>0.8</mu1>
+    <mu2>0.05</mu2>
+    <kp>1000000.0</kp>
+    <kd>100.0</kd>
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