Commit message: added SLAM

File: src/rover_description/urdf/rover_with_control.xacro (robot description, xacro)
@@ -95,5 +95,5 @@
 </link>
 <!-- ============================================================== -->
-<!-- WHEELS - CORRECTED WITH LIMIT TAGS FOR DIFFDRIVE              -->
+<!-- WHEELS                                                         -->
 <!-- ============================================================== -->
 <!-- FRONT LEFT WHEEL -->
@@ -282,5 +282,4 @@
 <!-- RPLIDAR A1                                                     -->
 <!-- ============================================================== -->
-<!-- Lidar joint -->
 <joint name="lidar_joint" type="fixed">
     <origin xyz="0 0 ${lidar_mount_z}" rpy="0 0 0"/>
@@ -288,5 +287,4 @@
     <child link="lidar_link"/>
 </joint>
-<!-- Lidar link -->
 <link name="lidar_link">
     <visual name="lidar_body">
@@ -323,46 +321,5 @@
 </link>
 <!-- ============================================================== -->
-<!-- GAZEBO CONFIGURATIONS - ROS2 JAZZY COMPATIBLE                 -->
-<!-- ============================================================== -->
-<!-- Wheel Physics Properties -->
-<gazebo reference="front_left_wheel">
-    <mu1>0.8</mu1>
-    <mu2>0.05</mu2>
-    <kp>1000000.0</kp>
-    <kd>100.0</kd>
-    <minDepth>0.001</minDepth>
-    <material>Gazebo/DarkGrey</material>
-</gazebo>
-<gazebo reference="front_right_wheel">
-    <mu1>0.8</mu1>
-    <mu2>0.05</mu2>
-    <kp>1000000.0</kp>
-    <kd>100.0</kd>
-    <minDepth>0.001</minDepth>
-    <material>Gazebo/DarkGrey</material>
-</gazebo>
-<gazebo reference="rear_left_wheel">
-    <mu1>0.8</mu1>
-    <mu2>0.05</mu2>
-    <kp>1000000.0</kp>
-    <kd>100.0</kd>
-    <minDepth>0.001</minDepth>
-    <material>Gazebo/DarkGrey</material>
-</gazebo>
-<gazebo reference="rear_right_wheel">
-    <mu1>0.8</mu1>
-    <mu2>0.05</mu2>
-    <kp>1000000.0</kp>
-    <kd>100.0</kd>
-    <minDepth>0.001</minDepth>
-    <material>Gazebo/DarkGrey</material>
-</gazebo>
-<gazebo reference="base_link">
-    <mu1>0.2</mu1>
-    <mu2>0.2</mu2>
-    <material>Gazebo/Black</material>
-</gazebo>
-<!-- ============================================================== -->
-<!-- LIDAR SENSOR - GPU LIDAR (ROS2 JAZZY COMPATIBLE)              -->
+<!-- GAZEBO LIDAR SENSOR - RAYS FROM TOP                            -->
 <!-- ============================================================== -->
 <gazebo reference="lidar_link">
@@ -373,8 +330,4 @@
         <update_rate>10</update_rate>
         <topic>scan</topic>
-        <ros>
-            <namespace>/</namespace>
-            <remapping>scan:=/scan</remapping>
-        </ros>
         <frame_name>lidar_link</frame_name>
         <lidar>
@@ -407,5 +360,45 @@
 </gazebo>
 <!-- ============================================================== -->
-<!-- SENSORS SYSTEM PLUGIN - ROS2 JAZZY                            -->
+<!-- GAZEBO CONFIGURATIONS                                          -->
+<!-- ============================================================== -->
+<gazebo reference="front_left_wheel">
+    <mu1>0.8</mu1>
+    <mu2>0.05</mu2>
+    <kp>1000000.0</kp>
+    <kd>100.0</kd>
+    <minDepth>0.001</minDepth>
+    <material>Gazebo/DarkGrey</material>
+</gazebo>
+<gazebo reference="front_right_wheel">
+    <mu1>0.8</mu1>
+    <mu2>0.05</mu2>
+    <kp>1000000.0</kp>
+    <kd>100.0</kd>
+    <minDepth>0.001</minDepth>
+    <material>Gazebo/DarkGrey</material>
+</gazebo>
+<gazebo reference="rear_left_wheel">
+    <mu1>0.8</mu1>
+    <mu2>0.05</mu2>
+    <kp>1000000.0</kp>
+    <kd>100.0</kd>
+    <minDepth>0.001</minDepth>
+    <material>Gazebo/DarkGrey</material>
+</gazebo>
+<gazebo reference="rear_right_wheel">
+    <mu1>0.8</mu1>
+    <mu2>0.05</mu2>
+    <kp>1000000.0</kp>
+    <kd>100.0</kd>
+    <minDepth>0.001</minDepth>
+    <material>Gazebo/DarkGrey</material>
+</gazebo>
+<gazebo reference="base_link">
+    <mu1>0.2</mu1>
+    <mu2>0.2</mu2>
+    <material>Gazebo/Black</material>
+</gazebo>
+<!-- ============================================================== -->
+<!-- SENSORS SYSTEM PLUGIN                                         -->
 <!-- ============================================================== -->
 <gazebo>
@@ -417,73 +410,11 @@
 </gazebo>
 <!-- ============================================================== -->
-<!-- DIFFERENTIAL DRIVE PLUGIN - GAZEBO HARMONIC                   -->
+<!-- ROS2 CONTROL PLUGIN - THIS PROVIDES ODOMETRY                  -->
 <!-- ============================================================== -->
 <gazebo>
-    <plugin filename="gz-sim-diff-drive-system" name="gz::sim::systems::DiffDrive">
-        <!-- Left wheels -->
-        <left_joint>front_left_wheel_joint</left_joint>
-        <left_joint>rear_left_wheel_joint</left_joint>
-        <!-- Right wheels -->
-        <right_joint>front_right_wheel_joint</right_joint>
-        <right_joint>rear_right_wheel_joint</right_joint>
-        <!-- Wheel parameters -->
-        <wheel_separation>0.428</wheel_separation>
-        <wheel_radius>0.035</wheel_radius>
-        <!-- Velocity limits -->
-        <linear_velocity>2.0</linear_velocity>
-        <angular_velocity>2.0</angular_velocity>
-        <linear_acceleration>1.0</linear_acceleration>
-        <angular_acceleration>2.0</angular_acceleration>
-        <!-- Topics -->
-        <topic>cmd_vel</topic>
-        <odom_topic>odom</odom_topic>
-        <!-- Frames -->
-        <odom_frame>odom</odom_frame>
-        <frame_id>odom</frame_id>
-        <child_frame_id>base_footprint</child_frame_id>
-        <!-- Odometry configuration -->
-        <odom_publish_frequency>50</odom_publish_frequency>
-        <publish_odom>true</publish_odom>
-        <publish_odom_tf>true</publish_odom_tf>
+    <plugin filename="gz-ros2-control-system" name="gz::ros2_control::GazeboSimSystem">
+        <parameters>$(find rover_description)/config/controller.yaml</parameters>
+        <use_sim_time>true</use_sim_time>
     </plugin>
 </gazebo>
-<!-- ============================================================== -->
-<!-- ROS-GZ BRIDGE - SINGLE PLUGIN FOR ALL BRIDGES                 -->
-<!-- ============================================================== -->
-<gazebo>
-    <plugin
-        filename="gz-sim-ros-gz-bridge-system"
-        name="gz::sim::systems::RosGzBridge">
-        <config>
-            <!-- cmd_vel: ROS -> GZ (for controlling robot) -->
-            <bridge>
-                <topic>/cmd_vel</topic>
-                <gz_type>gz.msgs.Twist</gz_type>
-                <ros_type>geometry_msgs/msg/Twist</ros_type>
-                <direction>ROS_TO_GZ</direction>
-            </bridge>
-            <!-- odom: GZ -> ROS (for odometry) -->
-            <bridge>
-                <topic>/odom</topic>
-                <gz_type>gz.msgs.Odometry</gz_type>
-                <ros_type>nav_msgs/msg/Odometry</ros_type>
-                <direction>GZ_TO_ROS</direction>
-            </bridge>
-            <!-- scan: GZ -> ROS (for lidar) -->
-            <bridge>
-                <topic>/scan</topic>
-                <gz_type>gz.msgs.LaserScan</gz_type>
-                <ros_type>sensor_msgs/msg/LaserScan</ros_type>
-                <direction>GZ_TO_ROS</direction>
-            </bridge>
-            <!-- clock: GZ -> ROS (for sim time) -->
-            <bridge>
-                <topic>/clock</topic>
-                <gz_type>gz.msgs.Clock</gz_type>
-                <ros_type>rosgraph_msgs/msg/Clock</ros_type>
-                <direction>GZ_TO_ROS</direction>
-            </bridge>
-        </config>
-    </plugin>
-</gazebo>
 </robot>
